File: schematics/power-12VAC-5DC-7805.brd (EAGLE design)
At the start: 20.3 x 43.2 mm, 10 parts, among them IC1 7805TV

Commit message: power-supply: better components placement on stripboard
Parts:
- added GND1: WIREPAD2,15/1,0, wirepad:2,15/1,0
- moved IC1 7.62 mm to (5.08, 40.6)
- moved C2 2.54 mm to (2.54, 27.9)
- moved C3 2.54 mm to (8.89, 27.9)
- moved B1 2.54 mm to (5.08, 12.7)
- moved C1 2.54 mm to (3.81, 22.9)
- moved C4 2.54 mm to (7.62, 22.9)
Connections:
- net GND: now also GND1.1
Routing:
- net GND: track 47.4 -> 69.6 mm, vias 6 -> 15
- net VCC: track 29.0 -> 36.6 mm, vias 6 -> 8
- net N$25: track 5.08 -> 0.00 mm
- net N$24: track 5.08 -> 0.00 mm
- net N$18: track 5.08 -> 0.00 mm
- net N$17: track 5.08 -> 0.00 mm
- net N$11: track 5.08 -> 0.00 mm
- net N$10: track 5.08 -> 0.00 mm
- net N$19: track 5.08 -> 0.00 mm
- net N$16: track 5.08 -> 0.00 mm
- net N$1: track 17.8 -> 22.9 mm, vias 3 -> 5
- net -12V: track 5.08 -> 7.61 mm, vias 0 -> 2
- net +12V: track 11.2 -> 13.8 mm, vias 2 -> 3
Other:
- board size 20.3 x 43.2 mm -> 20.3 x 45.7 mm

Commit message: power supply: new stripboard layout
Parts:
- removed GND1: WIREPAD2,15/1,0, wirepad:2,15/1,0
- moved C4 15.5 mm to (10.2, 7.62), turned to 180 degrees
- moved C2 10.2 mm to (2.54, 17.8)
- moved C3 3.59 mm to (6.35, 30.5), turned to 0 degrees
Connections:
- net GND: no longer GND1.1
Routing:
- net GND: track 69.6 -> 36.6 mm, vias 15 -> 8
- net N$1: track 22.9 -> 33.0 mm, vias 5 -> 6
- net VCC: vias 8 -> 7
