File: schematics/power-12VAC-5DC-7805.sch (EAGLE design)
At the start: 6 parts, among them IC1 7805TV

Commit message: schematics: add wiredpads
Parts:
- added +12VAC, -12VAC, GND, VOUT: WIREPAD2,54/1,0, wirepad:WIREPAD2,54/1,0
Connections:
- net +12V: now also +12VAC.P
- net -12V: now also -12VAC.P
- net GND: now also GND.P
- net VCC: now also VOUT.P
Changed lines of the file:
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@@
 <part name="P+1" library="supply1" deviceset="+12V" device=""/>
 <part name="P-1" library="supply1" deviceset="-12V" device=""/>
+<part name="+12VAC" library="wirepad" deviceset="WIREPAD" device="2,54/1,0"/>
+<part name="-12VAC" library="wirepad" deviceset="WIREPAD" device="2,54/1,0"/>
+<part name="VOUT" library="wirepad" deviceset="WIREPAD" device="2,54/1,0"/>
+<part name="GND" library="wirepad" deviceset="WIREPAD" device="2,54/1,0"/>
 </parts>
 <sheets>
@@
 <instance part="P+1" gate="1" x="0" y="81.28"/>
 <instance part="P-1" gate="1" x="0" y="60.96"/>
+<instance part="+12VAC" gate="G$1" x="0" y="40.64" smashed="yes">
+<attribute name="NAME" x="-1.143" y="42.4942" size="1.778" layer="95"/>
+</instance>
+<instance part="-12VAC" gate="G$1" x="0" y="35.56" smashed="yes">
+<attribute name="NAME" x="-1.143" y="37.4142" size="1.778" layer="95"/>
+</instance>
+<instance part="VOUT" gate="G$1" x="0" y="30.48" smashed="yes">
+<attribute name="NAME" x="-1.143" y="32.3342" size="1.778" layer="95"/>
+</instance>
+<instance part="GND" gate="G$1" x="0" y="25.4" smashed="yes">
+<attribute name="NAME" x="-1.143" y="27.2542" size="1.778" layer="95"/>
+</instance>
 </instances>
 <busses>
@@
 <junction x="76.2" y="50.8"/>
 </segment>
+<segment>
+<pinref part="GND" gate="G$1" pin="P"/>
+<wire x1="2.54" y1="25.4" x2="5.08" y2="25.4" width="0.1524" layer="91"/>
+<label x="5.08" y="25.4" size="1.6764" layer="95" xref="yes"/>
+</segment>
 </net>
 <net name="VCC" class="0">
@@
 <label x="83.82" y="71.12" size="1.778" layer="95" xref="yes"/>
 </segment>
+<segment>
+<pinref part="VOUT" gate="G$1" pin="P"/>
+<wire x1="2.54" y1="30.48" x2="5.08" y2="30.48" width="0.1524" layer="91"/>
+<label x="5.08" y="30.48" size="1.6764" layer="95" xref="yes"/>
+</segment>
 </net>
 <net name="+12V" class="0">
@@
 <pinref part="B1" gate="1" pin="AC1"/>
 <wire x1="0" y1="76.2" x2="17.78" y2="76.2" width="0.1524" layer="91"/>
+</segment>
+<segment>
+<pinref part="+12VAC" gate="G$1" pin="P"/>
+<wire x1="2.54" y1="40.64" x2="5.08" y2="40.64" width="0.1524" layer="91"/>
+<label x="5.08" y="40.64" size="1.6764" layer="95" xref="yes"/>
 </segment>
 </net>
@@
 <wire x1="0" y1="66.04" x2="0" y2="63.5" width="0.1524" layer="91"/>
 </segment>
+<segment>
+<pinref part="-12VAC" gate="G$1" pin="P"/>
+<wire x1="2.54" y1="35.56" x2="5.08" y2="35.56" width="0.1524" layer="91"/>
+<label x="5.08" y="35.56" size="1.6764" layer="95" xref="yes"/>
+</segment>
 </net>

Commit message: schematics: wiring power supply on protoboard
Parts:
- removed +12VAC, -12VAC, VOUT: WIREPAD2,54/1,0, wirepad:WIREPAD2,54/1,0
- added +12~, +5V, -12~: WIREPAD2,15/1,0, wirepad:WIREPAD2,15/1,0
- C2, C4: device SparkFun-Capacitors:CAPPTH1 -> SparkFun-Capacitors:CAPPTH
- GND: value WIREPAD2,54/1,0 -> WIREPAD2,15/1,0; device wirepad:WIREPAD2,54/1,0 -> wirepad:WIREPAD2,15/1,0
Connections:
- net +12V: now also +12~.P; no longer +12VAC.P
- net -12V: now also -12~.P; no longer -12VAC.P
- net VCC: now also +5V.P; no longer VOUT.P
Changed lines of the file:
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@@
 <setting verticaltext="up"/>
 </settings>
-<grid distance="0.1" unitdist="inch" unit="inch" style="lines" multiple="1" display="yes" altdistance="0.01" altunitdist="inch" altunit="inch"/>
+<grid distance="0.1" unitdist="inch" unit="inch" style="lines" multiple="1" display="no" altdistance="0.01" altunitdist="inch" altunit="inch"/>
 <layers>
-<layer number="1" name="Top" color="4" fill="1" visible="no" active="no"/>
-<layer number="16" name="Bottom" color="1" fill="1" visible="no" active="no"/>
-<layer number="17" name="Pads" color="2" fill="1" visible="no" active="no"/>
-<layer number="18" name="Vias" color="2" fill="1" visible="no" active="no"/>
-<layer number="19" name="Unrouted" color="6" fill="1" visible="no" active="no"/>
-<layer number="20" name="Dimension" color="15" fill="1" visible="no" active="no"/>
-<layer number="21" name="tPlace" color="7" fill="1" visible="no" active="no"/>
-<layer number="22" name="bPlace" color="7" fill="1" visible="no" active="no"/>
-<layer number="23" name="tOrigins" color="15" fill="1" visible="no" active="no"/>
-<layer number="24" name="bOrigins" color="15" fill="1" visible="no" active="no"/>
-<layer number="25" name="tNames" color="7" fill="1" visible="no" active="no"/>
-<layer number="26" name="bNames" color="7" fill="1" visible="no" active="no"/>
-<layer number="27" name="tValues" color="7" fill="1" visible="no" active="no"/>
-<layer number="28" name="bValues" color="7" fill="1" visible="no" active="no"/>
+<layer number="1" name="Top" color="4" fill="1" visible="yes" active="no"/>
+<layer number="16" name="Bottom" color="1" fill="1" visible="yes" active="no"/>
+<layer number="17" name="Pads" color="2" fill="1" visible="yes" active="no"/>
+<layer number="18" name="Vias" color="2" fill="1" visible="yes" active="no"/>
+<layer number="19" name="Unrouted" color="6" fill="1" visible="yes" active="no"/>
+<layer number="20" name="Dimension" color="15" fill="1" visible="yes" active="no"/>
+<layer number="21" name="tPlace" color="7" fill="1" visible="yes" active="no"/>
+<layer number="22" name="bPlace" color="7" fill="1" visible="yes" active="no"/>
+<layer number="23" name="tOrigins" color="15" fill="1" visible="yes" active="no"/>
+<layer number="24" name="bOrigins" color="15" fill="1" visible="yes" active="no"/>
+<layer number="25" name="tNames" color="7" fill="1" visible="yes" active="no"/>
+<layer number="26" name="bNames" color="7" fill="1" visible="yes" active="no"/>
+<layer number="27" name="tValues" color="7" fill="1" visible="yes" active="no"/>
+<layer number="28" name="bValues" color="7" fill="1" visible="yes" active="no"/>
 <layer number="29" name="tStop" color="7" fill="3" visible="no" active="no"/>
 <layer number="30" name="bStop" color="7" fill="6" visible="no" active="no"/>
@@
 <layer number="35" name="tGlue" color="7" fill="4" visible="no" active="no"/>
 <layer number="36" name="bGlue" color="7" fill="5" visible="no" active="no"/>
-<layer number="37" name="tTest" color="7" fill="1" visible="no" active="no"/>
-<layer number="38" name="bTest" color="7" fill="1" visible="no" active="no"/>
+<layer number="37" name="tTest" color="7" fill="1" visible="yes" active="no"/>
+<layer number="38" name="bTest" color="7" fill="1" visible="yes" active="no"/>
 <layer number="39" name="tKeepout" color="4" fill="11" visible="no" active="no"/>
 <layer number="40" name="bKeepout" color="1" fill="11" visible="no" active="no"/>
@@
 <layer number="44" name="Drills" color="7" fill="1" visible="no" active="no"/>
 <layer number="45" name="Holes" color="7" fill="1" visible="no" active="no"/>
-<layer number="46" name="Milling" color="3" fill="1" visible="no" active="no"/>
-<layer number="47" name="Measures" color="7" fill="1" visible="no" active="no"/>
-<layer number="48" name="Document" color="7" fill="1" visible="no" active="no"/>
-<layer number="49" name="Reference" color="7" fill="1" visible="no" active="no"/>
-<layer number="50" name="dxf" color="7" fill="1" visible="no" active="no"/>
-<layer number="51" name="tDocu" color="6" fill="1" visible="no" active="no"/>
-<layer number="52" name="bDocu" color="7" fill="1" visible="no" active="no"/>
-<layer number="53" name="tGND_GNDA" color="7" fill="9" visible="no" active="no"/>
-<layer number="54" name="bGND_GNDA" color="1" fill="9" visible="no" active="no"/>
-<layer number="56" name="wert" color="7" fill="1" visible="no" active="no"/>
+<layer number="46" name="Milling" color="3" fill="1" visible="yes" active="no"/>
+<layer number="47" name="Measures" color="7" fill="1" visible="yes" active="no"/>
+<layer number="48" name="Document" color="7" fill="1" visible="yes" active="no"/>
+<layer number="49" name="Reference" color="7" fill="1" visible="yes" active="no"/>
+<layer number="50" name="dxf" color="7" fill="1" visible="yes" active="no"/>
+<layer number="51" name="tDocu" color="7" fill="1" visible="yes" active="no"/>
+<layer number="52" name="bDocu" color="7" fill="1" visible="yes" active="no"/>
+<layer number="53" name="tGND_GNDA" color="7" fill="9" visible="yes" active="no"/>
+<layer number="54" name="bGND_GNDA" color="1" fill="9" visible="yes" active="no"/>
+<layer number="56" name="wert" color="7" fill="1" visible="yes" active="no"/>
 <layer number="90" name="Modules" color="5" fill="1" visible="yes" active="yes"/>
 <layer number="91" name="Nets" color="2" fill="1" visible="yes" active="yes"/>
@@
 <part name="C1" library="SparkFun-Capacitors" deviceset="CAP_POL" device="PTH1" value="100uF"/>
 <part name="C3" library="SparkFun-Capacitors" deviceset="CAP_POL" device="PTH1" value="10uF"/>
-<part name="C2" library="SparkFun-Capacitors" deviceset="CAP" device="PTH1" value="33nF"/>
-<part name="C4" library="SparkFun-Capacitors" deviceset="CAP" device="PTH1" value="100nF"/>
+<part name="C2" library="SparkFun-Capacitors" deviceset="CAP" device="PTH" value="33nF"/>
+<part name="C4" library="SparkFun-Capacitors" deviceset="CAP" device="PTH" value="100nF"/>
 <part name="P+1" library="supply1" deviceset="+12V" device=""/>
 <part name="P-1" library="supply1" deviceset="-12V" device=""/>
-<part name="+12VAC" library="wirepad" deviceset="WIREPAD" device="2,54/1,0"/>
-<part name="-12VAC" library="wirepad" deviceset="WIREPAD" device="2,54/1,0"/>
-<part name="VOUT" library="wirepad" deviceset="WIREPAD" device="2,54/1,0"/>
-<part name="GND" library="wirepad" deviceset="WIREPAD" device="2,54/1,0"/>
+<part name="+12~" library="wirepad" deviceset="WIREPAD" device="2,15/1,0" value="WIREPAD2,15/1,0"/>
+<part name="-12~" library="wirepad" deviceset="WIREPAD" device="2,15/1,0" value="WIREPAD2,15/1,0"/>
+<part name="+5V" library="wirepad" deviceset="WIREPAD" device="2,15/1,0" value="WIREPAD2,15/1,0"/>
+<part name="GND" library="wirepad" deviceset="WIREPAD" device="2,15/1,0" value="WIREPAD2,15/1,0"/>
 </parts>
 <sheets>
@@
 <instance part="P+1" gate="1" x="0" y="81.28"/>
 <instance part="P-1" gate="1" x="0" y="60.96"/>
-<instance part="+12VAC" gate="G$1" x="0" y="40.64" smashed="yes">
+<instance part="+12~" gate="G$1" x="0" y="40.64" smashed="yes">
 <attribute name="NAME" x="-1.143" y="42.4942" size="1.778" layer="95"/>
 </instance>
-<instance part="-12VAC" gate="G$1" x="0" y="35.56" smashed="yes">
+<instance part="-12~" gate="G$1" x="0" y="35.56" smashed="yes">
 <attribute name="NAME" x="-1.143" y="37.4142" size="1.778" layer="95"/>
 </instance>
-<instance part="VOUT" gate="G$1" x="0" y="30.48" smashed="yes">
+<instance part="+5V" gate="G$1" x="0" y="30.48" smashed="yes">
 <attribute name="NAME" x="-1.143" y="32.3342" size="1.778" layer="95"/>
 </instance>
@@
 </segment>
 <segment>
-<pinref part="VOUT" gate="G$1" pin="P"/>
+<pinref part="+5V" gate="G$1" pin="P"/>
 <wire x1="2.54" y1="30.48" x2="5.08" y2="30.48" width="0.1524" layer="91"/>
 <label x="5.08" y="30.48" size="1.6764" layer="95" xref="yes"/>
@@
 </segment>
 <segment>
-<pinref part="+12VAC" gate="G$1" pin="P"/>
+<pinref part="+12~" gate="G$1" pin="P"/>
 <wire x1="2.54" y1="40.64" x2="5.08" y2="40.64" width="0.1524" layer="91"/>
 <label x="5.08" y="40.64" size="1.6764" layer="95" xref="yes"/>
@@
 </segment>
 <segment>
-<pinref part="-12VAC" gate="G$1" pin="P"/>
+<pinref part="-12~" gate="G$1" pin="P"/>
 <wire x1="2.54" y1="35.56" x2="5.08" y2="35.56" width="0.1524" layer="91"/>
 <label x="5.08" y="35.56" size="1.6764" layer="95" xref="yes"/>

Commit message: power-supply: better components placement on stripboard
Parts:
- added GND1: WIREPAD2,15/1,0, wirepad:WIREPAD2,15/1,0
Connections:
- net GND: now also GND1.P
Changed lines of the file:
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@@
 <grid distance="0.1" unitdist="inch" unit="inch" style="lines" multiple="1" display="no" altdistance="0.01" altunitdist="inch" altunit="inch"/>
 <layers>
-<layer number="1" name="Top" color="4" fill="1" visible="yes" active="no"/>
-<layer number="16" name="Bottom" color="1" fill="1" visible="yes" active="no"/>
-<layer number="17" name="Pads" color="2" fill="1" visible="yes" active="no"/>
-<layer number="18" name="Vias" color="2" fill="1" visible="yes" active="no"/>
-<layer number="19" name="Unrouted" color="6" fill="1" visible="yes" active="no"/>
-<layer number="20" name="Dimension" color="15" fill="1" visible="yes" active="no"/>
-<layer number="21" name="tPlace" color="7" fill="1" visible="yes" active="no"/>
-<layer number="22" name="bPlace" color="7" fill="1" visible="yes" active="no"/>
-<layer number="23" name="tOrigins" color="15" fill="1" visible="yes" active="no"/>
-<layer number="24" name="bOrigins" color="15" fill="1" visible="yes" active="no"/>
-<layer number="25" name="tNames" color="7" fill="1" visible="yes" active="no"/>
-<layer number="26" name="bNames" color="7" fill="1" visible="yes" active="no"/>
-<layer number="27" name="tValues" color="7" fill="1" visible="yes" active="no"/>
-<layer number="28" name="bValues" color="7" fill="1" visible="yes" active="no"/>
+<layer number="1" name="Top" color="4" fill="1" visible="no" active="no"/>
+<layer number="16" name="Bottom" color="1" fill="1" visible="no" active="no"/>
+<layer number="17" name="Pads" color="2" fill="1" visible="no" active="no"/>
+<layer number="18" name="Vias" color="2" fill="1" visible="no" active="no"/>
+<layer number="19" name="Unrouted" color="6" fill="1" visible="no" active="no"/>
+<layer number="20" name="Dimension" color="15" fill="1" visible="no" active="no"/>
+<layer number="21" name="tPlace" color="7" fill="1" visible="no" active="no"/>
+<layer number="22" name="bPlace" color="7" fill="1" visible="no" active="no"/>
+<layer number="23" name="tOrigins" color="15" fill="1" visible="no" active="no"/>
+<layer number="24" name="bOrigins" color="15" fill="1" visible="no" active="no"/>
+<layer number="25" name="tNames" color="7" fill="1" visible="no" active="no"/>
+<layer number="26" name="bNames" color="7" fill="1" visible="no" active="no"/>
+<layer number="27" name="tValues" color="7" fill="1" visible="no" active="no"/>
+<layer number="28" name="bValues" color="7" fill="1" visible="no" active="no"/>
 <layer number="29" name="tStop" color="7" fill="3" visible="no" active="no"/>
 <layer number="30" name="bStop" color="7" fill="6" visible="no" active="no"/>
@@
 <layer number="35" name="tGlue" color="7" fill="4" visible="no" active="no"/>
 <layer number="36" name="bGlue" color="7" fill="5" visible="no" active="no"/>
-<layer number="37" name="tTest" color="7" fill="1" visible="yes" active="no"/>
-<layer number="38" name="bTest" color="7" fill="1" visible="yes" active="no"/>
+<layer number="37" name="tTest" color="7" fill="1" visible="no" active="no"/>
+<layer number="38" name="bTest" color="7" fill="1" visible="no" active="no"/>
 <layer number="39" name="tKeepout" color="4" fill="11" visible="no" active="no"/>
 <layer number="40" name="bKeepout" color="1" fill="11" visible="no" active="no"/>
@@
 <layer number="44" name="Drills" color="7" fill="1" visible="no" active="no"/>
 <layer number="45" name="Holes" color="7" fill="1" visible="no" active="no"/>
-<layer number="46" name="Milling" color="3" fill="1" visible="yes" active="no"/>
-<layer number="47" name="Measures" color="7" fill="1" visible="yes" active="no"/>
-<layer number="48" name="Document" color="7" fill="1" visible="yes" active="no"/>
-<layer number="49" name="Reference" color="7" fill="1" visible="yes" active="no"/>
-<layer number="50" name="dxf" color="7" fill="1" visible="yes" active="no"/>
-<layer number="51" name="tDocu" color="7" fill="1" visible="yes" active="no"/>
-<layer number="52" name="bDocu" color="7" fill="1" visible="yes" active="no"/>
-<layer number="53" name="tGND_GNDA" color="7" fill="9" visible="yes" active="no"/>
-<layer number="54" name="bGND_GNDA" color="1" fill="9" visible="yes" active="no"/>
-<layer number="56" name="wert" color="7" fill="1" visible="yes" active="no"/>
+<layer number="46" name="Milling" color="3" fill="1" visible="no" active="no"/>
+<layer number="47" name="Measures" color="7" fill="1" visible="no" active="no"/>
+<layer number="48" name="Document" color="7" fill="1" visible="no" active="no"/>
+<layer number="49" name="Reference" color="7" fill="1" visible="no" active="no"/>
+<layer number="50" name="dxf" color="7" fill="1" visible="no" active="no"/>
+<layer number="51" name="tDocu" color="7" fill="1" visible="no" active="no"/>
+<layer number="52" name="bDocu" color="7" fill="1" visible="no" active="no"/>
+<layer number="53" name="tGND_GNDA" color="7" fill="9" visible="no" active="no"/>
+<layer number="54" name="bGND_GNDA" color="1" fill="9" visible="no" active="no"/>
+<layer number="56" name="wert" color="7" fill="1" visible="no" active="no"/>
 <layer number="90" name="Modules" color="5" fill="1" visible="yes" active="yes"/>
 <layer number="91" name="Nets" color="2" fill="1" visible="yes" active="yes"/>
@@
 <part name="+5V" library="wirepad" deviceset="WIREPAD" device="2,15/1,0" value="WIREPAD2,15/1,0"/>
 <part name="GND" library="wirepad" deviceset="WIREPAD" device="2,15/1,0" value="WIREPAD2,15/1,0"/>
+<part name="GND1" library="wirepad" deviceset="WIREPAD" device="2,15/1,0" value="WIREPAD2,15/1,0"/>
 </parts>
 <sheets>
@@
 <instance part="GND" gate="G$1" x="0" y="25.4" smashed="yes">
 <attribute name="NAME" x="-1.143" y="27.2542" size="1.778" layer="95"/>
+</instance>
+<instance part="GND1" gate="G$1" x="0" y="20.32" smashed="yes">
+<attribute name="NAME" x="-1.143" y="22.1742" size="1.778" layer="95"/>
 </instance>
 </instances>
@@
 <label x="5.08" y="25.4" size="1.6764" layer="95" xref="yes"/>
 </segment>
+<segment>
+<pinref part="GND1" gate="G$1" pin="P"/>
+<wire x1="2.54" y1="20.32" x2="5.08" y2="20.32" width="0.1524" layer="91"/>
+<label x="5.08" y="20.32" size="1.6764" layer="95" xref="yes"/>
+</segment>
 </net>

Commit message: power supply: new stripboard layout
Parts:
- removed GND1: WIREPAD2,15/1,0, wirepad:WIREPAD2,15/1,0
Connections:
- net GND: no longer GND1.P
Changed lines of the file:
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@@
 <part name="+5V" library="wirepad" deviceset="WIREPAD" device="2,15/1,0" value="WIREPAD2,15/1,0"/>
 <part name="GND" library="wirepad" deviceset="WIREPAD" device="2,15/1,0" value="WIREPAD2,15/1,0"/>
-<part name="GND1" library="wirepad" deviceset="WIREPAD" device="2,15/1,0" value="WIREPAD2,15/1,0"/>
 </parts>
 <sheets>
@@
 <instance part="GND" gate="G$1" x="0" y="25.4" smashed="yes">
 <attribute name="NAME" x="-1.143" y="27.2542" size="1.778" layer="95"/>
-</instance>
-<instance part="GND1" gate="G$1" x="0" y="20.32" smashed="yes">
-<attribute name="NAME" x="-1.143" y="22.1742" size="1.778" layer="95"/>
 </instance>
 </instances>
@@
 <label x="5.08" y="25.4" size="1.6764" layer="95" xref="yes"/>
 </segment>
-<segment>
-<pinref part="GND1" gate="G$1" pin="P"/>
-<wire x1="2.54" y1="20.32" x2="5.08" y2="20.32" width="0.1524" layer="91"/>
-<label x="5.08" y="20.32" size="1.6764" layer="95" xref="yes"/>
-</segment>
 </net>
